File: stingyraycontrol9000.kicad_pcb (KiCad board)
At the start: 2 copper layers, 13 parts, among them J1 Screw_Terminal_01x04, J2 Screw_Terminal_01x04, J3 Screw_Terminal_01x02, J4 Conn_01x04, U1 ws2801, U2 LDD-L, U3 LDD-H

Commit message: remove third mounting hole
Parts:
- removed the J2 at (145.0, 147.3)
- removed the MK1 at (127.8, 90.4)
- added J1: Screw_Terminal_01x04, TerminalBlock_Phoenix:TerminalBlock_Phoenix_PT-1,5-4-5.0-H_1x04_P5.00mm_Horizontal, F.Cu at (145.0, 146.3)
- moved MK2 2.05 mm to (132.3, 135.6)
- moved J2 1.70 mm to (130.0, 69.1)
- renumbered J1 to J2, MK2 to MK1, MK3 to MK2
Changed lines of the file:
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@@
     (tracks 0)
     (zones 0)
-    (modules 13)
+    (modules 12)
     (nets 13)
   )
@@
   )
   (module MountingHole:MountingHole_3.2mm_M3_Pad (layer F.Cu)
-    (at 127.762 90.424)
+    (at 145.288 80.518)
     (descr "Mounting Hole 3.2mm, M3")
     (tags "mounting hole 3.2mm m3")
@@
       (effects (font (size 1 1) (thickness 0.15)))
     )
+    (fp_circle (center 0 0) (end 3.45 0) (layer F.CrtYd) (width 0.05))
+    (fp_circle (center 0 0) (end 3.2 0) (layer Cmts.User) (width 0.15))
     (fp_text user %R (at 0.3 0) (layer F.Fab)
       (effects (font (size 1 1) (thickness 0.15)))
     )
-    (fp_circle (center 0 0) (end 3.2 0) (layer Cmts.User) (width 0.15))
-    (fp_circle (center 0 0) (end 3.45 0) (layer F.CrtYd) (width 0.05))
     (pad 1 thru_hole circle (at 0 0) (size 6.4 6.4) (drill 3.2) (layers *.Cu *.Mask))
   )
   (module MountingHole:MountingHole_3.2mm_M3_Pad (layer F.Cu)
-    (at 145.288 80.518)
+    (at 132.334 135.636)
     (descr "Mounting Hole 3.2mm, M3")
     (tags "mounting hole 3.2mm m3")
     (attr virtual)
     (fp_text reference MK2 (at 0 -4.2) (layer F.SilkS)
-      (effects (font (size 1 1) (thickness 0.15)))
-    )
-    (fp_text value Mounting_Hole (at 0 4.2) (layer F.Fab)
-      (effects (font (size 1 1) (thickness 0.15)))
-    )
-    (fp_circle (center 0 0) (end 3.45 0) (layer F.CrtYd) (width 0.05))
-    (fp_circle (center 0 0) (end 3.2 0) (layer Cmts.User) (width 0.15))
-    (fp_text user %R (at 0.3 0) (layer F.Fab)
-      (effects (font (size 1 1) (thickness 0.15)))
-    )
-    (pad 1 thru_hole circle (at 0 0) (size 6.4 6.4) (drill 3.2) (layers *.Cu *.Mask))
-  )
-  (module MountingHole:MountingHole_3.2mm_M3_Pad (layer F.Cu)
-    (at 134.112 136.652)
-    (descr "Mounting Hole 3.2mm, M3")
-    (tags "mounting hole 3.2mm m3")
-    (attr virtual)
-    (fp_text reference MK3 (at 0 -4.2) (layer F.SilkS)
       (effects (font (size 1 1) (thickness 0.15)))
     )
@@
   (module meanwell_led_driver:LDD_L (layer F.Cu)
     (at 137.6172 112.4966 270)
-    (fp_text reference U2 (at 0 -2.54 270) (layer F.SilkS)
+    (fp_text reference U2 (at -6.0706 -2.8448) (layer F.SilkS)
       (effects (font (size 1 1) (thickness 0.15)))
     )
@@
   (module meanwell_led_driver:LDD_H (layer F.Cu)
     (at 137.668 112.522)
-    (fp_text reference U3 (at 0 -1.27) (layer F.SilkS)
+    (fp_text reference U3 (at -8.128 -8.382) (layer F.SilkS)
       (effects (font (size 1 1) (thickness 0.15)))
     )
@@
   )
   (module TerminalBlock_Phoenix:TerminalBlock_Phoenix_PT-1,5-4-5.0-H_1x04_P5.00mm_Horizontal (layer F.Cu)
-    (at 129.286 67.564)
+    (at 130.048 69.088)
     (descr "Terminal Block Phoenix PT-1,5-4-5.0-H, 4 pins, pitch 5mm, size 20x9mm^2, drill diamater 1.3mm, pad diameter 2.6mm, see http://www.mouser.com/ds/2/324/ItemDetail_1935161-922578.pdf, script-generated using https://github.com/pointhi/kicad-footprint-generator/scripts/TerminalBlock_Phoenix")
     (tags "THT Terminal Block Phoenix PT-1,5-4-5.0-H pitch 5mm size 20x9mm^2 drill 1.3mm pad 2.6mm")
-    (fp_text reference J1 (at 7.5 -5.06) (layer F.SilkS)
+    (fp_text reference J2 (at 7.5 -5.06) (layer F.SilkS)
       (effects (font (size 1 1) (thickness 0.15)))
     )
@@
   )
   (module TerminalBlock_Phoenix:TerminalBlock_Phoenix_PT-1,5-4-5.0-H_1x04_P5.00mm_Horizontal (layer F.Cu)
-    (at 145.034 147.32 180)
+    (at 145.034 146.304 180)
     (descr "Terminal Block Phoenix PT-1,5-4-5.0-H, 4 pins, pitch 5mm, size 20x9mm^2, drill diamater 1.3mm, pad diameter 2.6mm, see http://www.mouser.com/ds/2/324/ItemDetail_1935161-922578.pdf, script-generated using https://github.com/pointhi/kicad-footprint-generator/scripts/TerminalBlock_Phoenix")
     (tags "THT Terminal Block Phoenix PT-1,5-4-5.0-H pitch 5mm size 20x9mm^2 drill 1.3mm pad 2.6mm")
-    (fp_text reference J2 (at 7.5 -5.06 180) (layer F.SilkS)
-      (effects (font (size 1 1) (thickness 0.15)))
-    )
+    (fp_text reference J1 (at 7.5 -5.06 180) (layer F.SilkS)
+      (effects (font (size 1 1) (thickness 0.15)))
+    )

Commit message: route board
Parts:
- MK1, MK2: footprint MountingHole:MountingHole_3.2mm_M3_Pad -> MountingHole:MountingHole_3.2mm_M3
- moved MK2 2.30 mm to (130.0, 135.9)
- moved J2 1.02 mm to (130.0, 70.1)
- moved C1 0.51 mm to (138.9, 84.6)
- moved D1 0.51 mm to (138.9, 81.3)
- moved R1 0.51 mm to (138.9, 78.0)
- moved U1 0.51 mm to (136.4, 90.9)
- moved MK1 0.25 mm to (145.0, 80.5)
Routing:
- net /CKO: track 0.00 -> 61.3 mm, vias 0 -> 1
- net /SDO: track 0.00 -> 59.1 mm, vias 0 -> 1
- net /ROUT: track 0.00 -> 29.5 mm
- net /SDI: track 0.00 -> 21.7 mm, vias 0 -> 1
- net /CKI: track 0.00 -> 18.4 mm, vias 0 -> 1
- net +5V: track 0.00 -> 17.4 mm
- net /GOUT: track 0.00 -> 7.79 mm
- net /BOUT: track 0.00 -> 7.27 mm
- net GND: vias 0 -> 8
- added copper zone on B.Cu, net +24V
- added copper zone on F.Cu, net /LED+
- added copper zone on F.Cu, net /LED-
- added copper zone on B.Cu, net GND
Other:
- board outline added: 22.1 x 86.4 mm
- net class Default: trace_width 0.25 -> 0.2
- net class data added: clearance 0.2, trace_width 0.2, via_dia 0.6, via_drill 0.3
- net class power added: clearance 0.2, trace_width 0.25, via_dia 0.8, via_drill 0.4
- board text added: "B"
- board text added: "CKI"
- board text added: "CKO"
- board text added: "G"
- board text added: "GND"
- board text added: "LED+"
- board text added: "LED-"
- board text added: "R"
- board text added: "SDI"
- board text added: "SDO"
- board text added: "VCC"
- board text added: "stingyraycontrol9000"

Commit message: slight optimizations
Parts:
- MK1, MK2: footprint MountingHole:MountingHole_3.2mm_M3 -> MountingHole:MountingHole_3.2mm_M3_ISO14580
- moved MK1 0.13 mm to (145.2, 80.5)
- moved MK2 0.13 mm to (129.9, 135.9)
Routing:
- net /ROUT: track 29.5 -> 34.5 mm
- net /CKO: track 61.3 -> 60.4 mm

Commit message: add logos to pcb
Parts:
- added G***: LOGO, logos:entropia, B.Cu at (137.9, 95.1)
- added G***: LOGO, logos:goethe, B.Cu at (143.8, 112.8)
- added G***: LOGO, logos:zkm, B.Cu at (129.3, 104.8)
Other:
- board text added: "built for »Open Codes. The Art of Coding«"
- board text added: "github.com/felixheld/ stingyraycontrol9000 CC BY-SA 4.0"
- board text added: "v1.0"
- board text removed: "stingyraycontrol9000"
